Commit message: Adding markers with changing colors

File: rhr_visualization/urdf/Hand_Assem.URDF (robot description, URDF)
Before this commit: robot Hand_Assem, 9 links, 8 joints
Links:
- added link /dist2_tactile
- added link dist1_tactile
- added link dist3_tactile
- added link prox1_tactile
- added link prox2_tactile
- added link prox3_tactile
Joints:
- added joint dist1_tactile_joint: type fixed, parent distal1, child dist1_tactile, origin xyz=0 0 0 rpy=3.1415 -1.5708 0
- added joint dist2_tactile_joint: type fixed, parent distal2, child /dist2_tactile, origin xyz=0 0 0 rpy=3.1415 -1.5708 0
- added joint dist3_tactile_joint: type fixed, parent distal3, child dist3_tactile, origin xyz=0 0 0 rpy=3.1415 -1.5708 0
- added joint prox1_tactile_joint: type fixed, parent proximal1, child prox1_tactile, origin xyz=0 0 0 rpy=0 -1.5708 0
- added joint prox2_tactile_joint: type fixed, parent proximal2, child prox2_tactile, origin xyz=0 0 0 rpy=0 -1.5708 0
- added joint prox3_tactile_joint: type fixed, parent proximal3, child prox3_tactile, origin xyz=0 0 0 rpy=0 -1.5708 0
