Commit message: Changed to the final CAD, not quite done

File: rhr_visualization/urdf/full_reflex_model.urdf.xacro (robot description, xacro)
@@ -14,8 +14,8 @@
  		<color rgba="0.22 0.22 0.22 1"/>
  	</xacro:macro>
- 	<xacro:macro name="prox_color">
+ 	<xacro:macro name="proximal_color">
  		<color rgba="0.35 0.35 0.35 1"/>
  	</xacro:macro>
- 	 <xacro:macro name="dist_color">
+ 	 <xacro:macro name="distal_color">
  		<color rgba="0.35 0.35 0.35 1"/>
  	</xacro:macro>
@@ -23,4 +23,7 @@
  		<color rgba="0.2 0.2 .2 1"/>
  	</xacro:macro>
+  <xacro:macro name="pad_color">
+    <color rgba="0.686 0.0706 0.8039 0.4"/>
+  </xacro:macro>
 	<!-- Macro to make each park of the link -->
 	<xacro:macro name="flex_link" params="finger_id flex_id">
@@ -48,5 +51,5 @@
 	<xacro:macro name="flex_to_segment_joint" params="finger_id">
 		<joint name="finger[${finger_id}]/flex_joint_from_prox_to_1" type="continuous">
-			<parent link="proximal${finger_id}"/>
+			<parent link="proximal_${finger_id}"/>
 			<child link="finger[${finger_id}]/flex_link[1]"/>
 			<origin xyz="${prox_length} 0 0.003"/>
@@ -55,5 +58,5 @@
 		<joint name="finger[${finger_id}]/flex_joint_from_${num_steps}_to_dist" type="continuous">
 			<parent link="finger[${finger_id}]/flex_link[${num_steps}]"/>
-			<child link="distal${finger_id}"/>
+			<child link="distal_${finger_id}"/>
 			<origin xyz="${flex_length/num_steps-0.01} 0 0.003"/>
 			<axis xyz="0 -1 0"/>
@@ -91,18 +94,49 @@
   <link
     name="base_link">
-    <inertial>
-      <origin
-        xyz="3.0216E-05 -0.010622 -0.0169"
+    <visual>
+      <origin
+        xyz="0 0 0"
         rpy="0 0 0" />
-      <mass
-        value="0.24584" />
-      <inertia
-        ixx="0.00046643"
-        ixy="3.914E-07"
-        ixz="-1.1388E-06"
-        iyy="0.00036883"
-        iyz="-3.3676E-05"
-        izz="0.00046818" />
-    </inertial>
+      <geometry>
+        <mesh
+          filename="package://rhr_visualization/meshes/base_link.STL" />
+      </geometry>
+      <material
+        name="">
+          <xacro:base_color/>
+      </material>
+    </visual>
+  </link>
+  <link
+    name="pad">
+    <visual>
+      <origin
+        xyz="0 0 0"
+        rpy="${pi/2} 0 ${-pi/2}" />
+      <geometry>
+        <mesh
+          filename="package://rhr_visualization/meshes/pad.STL" />
+      </geometry>
+      <material
+        name="">
+        <xacro:pad_color/>
+      </material>
+    </visual>
+  </link>
+  <joint
+    name="pad_joint"
+    type="fixed">
+    <origin
+      xyz="0 0 0"
+      rpy="0 0 0" />
+    <parent
+      link="base_link" />
+    <child
+      link="pad" />
+    <axis
+      xyz="0 0 0" />
+  </joint>
+  <link
+    name="swivel_1">
     <visual>
       <origin
@@ -111,12 +145,28 @@
       <geometry>
         <mesh
-          filename="package://rhr_visualization/meshes/base_link.STL" />
-      </geometry>
-      <material
-        name="">
-        	<xacro:base_color/>
-      </material>
-    </visual>
-    <collision>
+          filename="package://rhr_visualization/meshes/swivel_1.STL" />
+      </geometry>
+      <material
+        name="">
+        <xacro:swivel_color/>
+      </material>
+    </visual>
+  </link>
+  <joint
+    name="preshape_1"
+    type="continuous">
+    <origin
+      xyz="0.0503973683071414 -0.026 0.063"
+      rpy="6.75550818663469E-16 1.97993848419069E-16 -2.77555756156289E-16" />
+    <parent
+      link="base_link" />
+    <child
+      link="swivel_1" />
+    <axis
+      xyz="0 0 -1" />
+  </joint>
+  <link
+    name="proximal_1">
+    <visual>
       <origin
         xyz="0 0 0"
@@ -124,24 +174,143 @@
       <geometry>
         <mesh
-          filename="package://rhr_visualization/meshes/base_link.STL" />
-      </geometry>
-    </collision>
-  </link>
-  <link
-    name="swivel1">
-    <inertial>
-      <origin
-        xyz="0.00017449 0.0052831 0.0054101"
+          filename="package://rhr_visualization/meshes/proximal_1.STL" />
+      </geometry>
+      <material
+        name="">
+        <xacro:proximal_color/>
+      </material>
+    </visual>
+  </link>
+  <joint
+    name="proximal_joint_1"
+    type="continuous">
+    <origin
+      xyz="0.01 0 0.0186"
+      rpy="-6.20039667432211E-16 2.40507565059625E-17 2.22044604925031E-16" />
+    <parent
+      link="swivel_1" />
+    <child
+      link="proximal_1" />
+    <axis
+      xyz="0 -1 0" />
+  </joint>
+  <link
+    name="proximal_pad_1">
+    <visual>
+      <origin
+        xyz="-0.065 0.026 -0.083"
+        rpy="${pi/2} 0 ${-pi/2}" />
+      <geometry>
+        <mesh
+          filename="package://rhr_visualization/meshes/proximal_pad_1.STL" />
+      </geometry>
+      <material
+        name="">
+        <xacro:pad_color/>
+      </material>
+    </visual>
+  </link>
+  <joint
+    name="proximal_1_pad_joint"
+    type="fixed">
+    <origin
+      xyz="0 0 0"
+      rpy="0 0 0" />
+    <parent
+      link="proximal_1" />
+    <child
+      link="proximal_pad_1" />
+    <axis
+      xyz="0 0 0" />
+  </joint>
+  <link
+    name="distal_1">
+    <visual>
+      <origin
+        xyz="-0.13 0.026 -0.088"
+        rpy="${pi/2} 0 ${-pi/2}" />
+      <geometry>
+        <mesh
+          filename="package://rhr_visualization/meshes/distal_1.STL" />
+      </geometry>
+      <material
+        name="">
+        <xacro:distal_color/>
+      </material>
+    </visual>
+  </link>
+<!--   <joint
+    name="distal_joint_1"
+    type="continuous">
+    <origin
+      xyz="0.0760000000000001 0 0.0025"
+      rpy="0 0 0" />
+    <parent
+      link="proximal_1" />
+    <child
+      link="distal_1" />
+    <axis
+      xyz="0 -1 0" />
+  </joint> -->
+  <link
+    name="distal_pad_1">
+    <visual>
+      <origin
+        xyz="-0.13 0.026 -0.088"
+        rpy="${pi/2} 0 ${-pi/2}" />
+      <geometry>
+        <mesh
+          filename="package://rhr_visualization/meshes/distal_pad_1.STL" />
+      </geometry>
+      <material
+        name="">
+        <xacro:pad_color/>
+      </material>
+    </visual>
+  </link>
+  <joint
+    name="distal_1_pad_joint"
+    type="fixed">
+    <origin
+      xyz="0 0 0"
+      rpy="0 0 0" />
+    <parent
+      link="distal_1" />
+    <child
+      link="distal_pad_1" />
+    <axis
+      xyz="0 0 0" />
+  </joint>
+  <link
+    name="swivel_2">
+    <visual>
+      <origin
+        xyz="0 0 0"
         rpy="0 0 0" />
-      <mass
-        value="0.012217" />
-      <inertia
-        ixx="1.6714E-06"
-        ixy="1.5123E-08"
-        ixz="9.7662E-09"
-        iyy="2.2057E-06"
-        iyz="3.9094E-07"
-        izz="2.216E-06" />
-    </inertial>
+      <geometry>
+        <mesh
+          filename="package://rhr_visualization/meshes/swivel_2.STL" />
+      </geometry>
+      <material
+        name="">
+        <xacro:swivel_color/>
+      </material>
+    </visual>
+  </link>
+  <joint
+    name="preshape_2"
+    type="continuous">
+    <origin
+      xyz="0.0503973683071413 0.0259999999999999 0.063"
+      rpy="1.22459340959228E-15 -7.33448407631817E-16 -1.66533453693773E-16" />
+    <parent
+      link="base_link" />
+    <child
+      link="swivel_2" />
+    <axis
+      xyz="0 0 -1" />
+  </joint>
+  <link
+    name="proximal_2">
     <visual>
       <origin
@@ -150,12 +319,115 @@
       <geometry>
         <mesh
-          filename="package://rhr_visualization/meshes/swivel1.STL" />
-      </geometry>
-      <material
-        name="">
-        <xacro:swivel_color/>
-      </material>
-    </visual>
-    <collision>
+          filename="package://rhr_visualization/meshes/proximal_2.STL" />
+      </geometry>
+      <material
+        name="">
+        <xacro:proximal_color/>
+      </material>
+    </visual>
+  </link>
+  <joint
+    name="proximal_joint_2"
+    type="continuous">
+    <origin
+      xyz="0.01 0 0.0186"
+      rpy="-1.16908225836102E-15 9.55493012556849E-16 1.11022302462515E-16" />
+    <parent
+      link="swivel_2" />
+    <child
+      link="proximal_2" />
+    <axis
+      xyz="0 -1 0" />
+  </joint>
+  <link
+    name="proximal_pad_2">
+    <visual>
+      <origin
+        xyz="-0.065 -0.026 -0.083"
+        rpy="${pi/2} 0 ${-pi/2}" />
+      <geometry>
+        <mesh
+          filename="package://rhr_visualization/meshes/proximal_pad_2.STL" />
+      </geometry>
+      <material
+        name="">
+        <xacro:pad_color/>
+      </material>
+    </visual>
+  </link>
+  <joint
+    name="proximal_2_pad_joint"
+    type="fixed">
+    <origin
+      xyz="0 0 0"
+      rpy="0 0 0" />
+    <parent
+      link="proximal_2" />
+    <child
+      link="proximal_pad_2" />
+    <axis
+      xyz="0 0 0" />
+  </joint>
+  <link
+    name="distal_2">
+    <visual>
+      <origin
+        xyz="-0.13 -0.026 -0.088"
+        rpy="${pi/2} 0 ${-pi/2}" />
+      <geometry>
+        <mesh
+          filename="package://rhr_visualization/meshes/distal_2.STL" />
+      </geometry>
+      <material
+        name="">
+        <xacro:distal_color/>
+      </material>
+    </visual>
+  </link>
+<!--   <joint
+    name="distal_joint_2"
+    type="continuous">
+    <origin
+      xyz="0.076 0 0.0025"
+      rpy="0 0 0" />
+    <parent
+      link="proximal_2" />
+    <child
+      link="distal_2" />
+    <axis
+      xyz="0 -1 0" />
+  </joint> -->
+  <link
+    name="distal_pad_2">
+    <visual>
+      <origin
+        xyz="-0.13 -0.026 -0.088"
+        rpy="${pi/2} 0 ${-pi/2}" />
+      <geometry>
+        <mesh
+          filename="package://rhr_visualization/meshes/distal_pad_2.STL" />
+      </geometry>
+      <material
+        name="">
+        <xacro:pad_color/>
+      </material>
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
Commit message: Folded in final CAD successfully

File: rhr_visualization/urdf/full_reflex_model.urdf.xacro (robot description, xacro)
@@ -104,5 +104,5 @@
       <material
         name="">
-          <xacro:base_color/>
+        <xacro:base_color/>
       </material>
     </visual>
@@ -113,5 +113,5 @@
       <origin
         xyz="0 0 0"
-        rpy="${pi/2} 0 ${-pi/2}" />
+        rpy="0 0 0" />
       <geometry>
         <mesh
@@ -128,6 +128,6 @@
     type="fixed">
     <origin
-      xyz="0 0 0"
-      rpy="0 0 0" />
+      xyz="0.02 0 0.063"
+      rpy="1.5707963267949 5.55111512312578E-17 -1.5707963267949" />
     <parent
       link="base_link" />
@@ -199,6 +199,6 @@
     <visual>
       <origin
-        xyz="-0.065 0.026 -0.083"
-        rpy="${pi/2} 0 ${-pi/2}" />
+        xyz="0 0 0"
+        rpy="0 0 0" />
       <geometry>
         <mesh
@@ -212,51 +212,51 @@
   </link>
   <joint
-    name="proximal_1_pad_joint"
+    name="prox1_pad_joint"
     type="fixed">
     <origin
       xyz="0 0 0"
+      rpy="1.5707963267949 0 -1.5707963267949" />
+    <parent
+      link="proximal_1" />
+    <child
+      link="proximal_pad_1" />
+    <axis
+      xyz="0 0 0" />
+  </joint>
+  <link
+    name="distal_1">
+    <visual>
+      <origin
+        xyz="0 0 0"
+        rpy="0 0 0" />
+      <geometry>
+        <mesh
+          filename="package://rhr_visualization/meshes/distal_1.STL" />
+      </geometry>
+      <material
+        name="">
+        <xacro:distal_color/>
+      </material>
+    </visual>
+  </link>
+  <joint
+    name="distal_joint_1"
+    type="continuous">
+    <origin
+      xyz="0.0760000000000001 0 0.00250000000000002"
       rpy="0 0 0" />
     <parent
       link="proximal_1" />
     <child
-      link="proximal_pad_1" />
-    <axis
-      xyz="0 0 0" />
-  </joint>
-  <link
-    name="distal_1">
-    <visual>
-      <origin
-        xyz="-0.13 0.026 -0.088"
-        rpy="${pi/2} 0 ${-pi/2}" />
-      <geometry>
-        <mesh
-          filename="package://rhr_visualization/meshes/distal_1.STL" />
-      </geometry>
-      <material
-        name="">
-        <xacro:distal_color/>
-      </material>
-    </visual>
-  </link>
-<!--   <joint
-    name="distal_joint_1"
-    type="continuous">
-    <origin
-      xyz="0.0760000000000001 0 0.0025"
-      rpy="0 0 0" />
-    <parent
-      link="proximal_1" />
-    <child
       link="distal_1" />
     <axis
       xyz="0 -1 0" />
-  </joint> -->
+  </joint>
   <link
     name="distal_pad_1">
     <visual>
       <origin
-        xyz="-0.13 0.026 -0.088"
-        rpy="${pi/2} 0 ${-pi/2}" />
+        xyz="0 0 0"
+        rpy="0 0 0" />
       <geometry>
         <mesh
@@ -270,9 +270,9 @@
   </link>
   <joint
-    name="distal_1_pad_joint"
-    type="fixed">
-    <origin
-      xyz="0 0 0"
-      rpy="0 0 0" />
+    name="dist1_pad_joint"
+    type="fixed">
+    <origin
+      xyz="-0.0760000000000001 0 -0.0025"
+      rpy="1.5707963267949 0 -1.5707963267949" />
     <parent
       link="distal_1" />
@@ -344,6 +344,6 @@
     <visual>
       <origin
-        xyz="-0.065 -0.026 -0.083"
-        rpy="${pi/2} 0 ${-pi/2}" />
+        xyz="0 0 0"
+        rpy="0 0 0" />
       <geometry>
         <mesh
@@ -357,25 +357,141 @@
   </link>
   <joint
-    name="proximal_2_pad_joint"
+    name="prox2_pad_joint"
     type="fixed">
     <origin
       xyz="0 0 0"
+      rpy="1.5707963267949 0 -1.5707963267949" />
+    <parent
+      link="proximal_2" />
+    <child
+      link="proximal_pad_2" />
+    <axis
+      xyz="0 0 0" />
+  </joint>
+  <link
+    name="distal_2">
+    <visual>
+      <origin
+        xyz="0 0 0"
+        rpy="0 0 0" />
+      <geometry>
+        <mesh
+          filename="package://rhr_visualization/meshes/distal_2.STL" />
+      </geometry>
+      <material
+        name="">
+        <xacro:distal_color/>
+      </material>
+    </visual>
+  </link>
+  <joint
+    name="distal_joint_2"
+    type="continuous">
+    <origin
+      xyz="0.0760000000000001 0 0.00249999999999997"
       rpy="0 0 0" />
     <parent
       link="proximal_2" />
     <child
-      link="proximal_pad_2" />
-    <axis
-      xyz="0 0 0" />
-  </joint>
-  <link
-    name="distal_2">
-    <visual>
-      <origin
-        xyz="-0.13 -0.026 -0.088"
-        rpy="${pi/2} 0 ${-pi/2}" />
-      <geometry>
-        <mesh
-          filename="package://rhr_visualization/meshes/distal_2.STL" />
+      link="distal_2" />
+    <axis
+      xyz="0 -1 0" />
+  </joint>
+  <link
+    name="distal_pad_2">
+    <visual>
+      <origin
+        xyz="0 0 0"
+        rpy="0 0 0" />
+      <geometry>
+        <mesh
+          filename="package://rhr_visualization/meshes/distal_pad_2.STL" />
+      </geometry>
+      <material
+        name="">
+        <xacro:pad_color/>
+      </material>
+    </visual>
+  </link>
+  <joint
+    name="dist2_pad_joint"
+    type="fixed">
+    <origin
+      xyz="-0.0760000000000001 0 -0.0025"
+      rpy="1.5707963267949 0 -1.5707963267949" />
+    <parent
+      link="distal_2" />
+    <child
+      link="distal_pad_2" />
+    <axis
+      xyz="0 0 0" />
+  </joint>
+  <link
+    name="proximal_3">
+    <visual>
+      <origin
+        xyz="0 0 0"
+        rpy="0 0 0" />
+      <geometry>
+        <mesh
+          filename="package://rhr_visualization/meshes/proximal_3.STL" />
+      </geometry>
+      <material
+        name="">
+        <xacro:proximal_color/>
+      </material>
+    </visual>
+  </link>
+  <joint
+    name="proximal_joint_3"
+    type="continuous">
+    <origin
+      xyz="-0.0299999999999996 0 0.0816000000000002"
+      rpy="-5.55111512312578E-17 -2.22044604925031E-16 3.14159265358979" />
+    <parent
+      link="base_link" />
+    <child
+      link="proximal_3" />
+    <axis
+      xyz="0 -1 0" />
+  </joint>
+  <link
+    name="proximal_pad_3">
+    <visual>
+      <origin
+        xyz="0 0 0"
+        rpy="0 0 0" />
+      <geometry>
+        <mesh
+          filename="package://rhr_visualization/meshes/proximal_pad_3.STL" />
+      </geometry>
+      <material
+        name="">
+        <xacro:pad_color/>
+      </material>
+    </visual>
+  </link>
+  <joint
+    name="prox3_pad_joint"
+    type="fixed">
+    <origin
+      xyz="0 0 0"
+      rpy="1.5707963267949 1.22460635382238E-16 -1.5707963267949" />
+    <parent
+      link="proximal_3" />
+    <child
+      link="proximal_pad_3" />
+    <axis
+      xyz="0 0 0" />
+  </joint>
+  <link
+    name="distal_3">
+    <visual>
+      <origin
+        xyz="0 0 0"
+        rpy="0 0 0" />
+      <geometry>
+        <mesh
+          filename="package://rhr_visualization/meshes/distal_3.STL" />
       </geometry>
       <material
@@ -385,139 +501,23 @@
     </visual>
   </link>
-<!--   <joint
-    name="distal_joint_2"
-    type="continuous">
-    <origin
-      xyz="0.076 0 0.0025"
-      rpy="0 0 0" />
-    <parent
-      link="proximal_2" />
-    <child
-      link="distal_2" />
+  <joint
+    name="distal_joint_3"
+    type="continuous">
+    <origin
+      xyz="0.0760000000000001 0 0.0025"
+      rpy="-1.48887961834512E-45 -1.0995850059156E-76 -7.38531841236285E-32" />
+    <parent
+      link="proximal_3" />
+    <child
+      link="distal_3" />
     <axis
       xyz="0 -1 0" />
-  </joint> -->
-  <link
-    name="distal_pad_2">
-    <visual>
-      <origin
-        xyz="-0.13 -0.026 -0.088"
-        rpy="${pi/2} 0 ${-pi/2}" />
-      <geometry>
-        <mesh
-          filename="package://rhr_visualization/meshes/distal_pad_2.STL" />
-      </geometry>
-      <material
-        name="">
-        <xacro:pad_color/>
-      </material>
-    </visual>
-  </link>
-  <joint
-    name="distal_2_pad_joint"
-    type="fixed">
-    <origin
-      xyz="0 0 0"
-      rpy="0 0 0" />
-    <parent
-      link="distal_2" />
-    <child
-      link="distal_pad_2" />
-    <axis
-      xyz="0 0 0" />
-  </joint>
-  <link
-    name="proximal_3">
-    <visual>
-      <origin
-        xyz="0 0 0"
-        rpy="0 0 0" />
-      <geometry>
-        <mesh
-          filename="package://rhr_visualization/meshes/proximal_3.STL" />
-      </geometry>
-      <material
-        name="">
-        <xacro:proximal_color/>
-      </material>
-    </visual>
-  </link>
-  <joint
-    name="proximal_joint_3"
-    type="continuous">
-    <origin
-      xyz="-0.03 0 0.0816000000000001"
-      rpy="-5.55111512312578E-17 -2.22044604925031E-16 3.14159265358979" />
-    <parent
-      link="base_link" />
-    <child
-      link="proximal_3" />
-    <axis
-      xyz="0 -1 0" />
-  </joint>
-  <link
-    name="proximal_pad_3">
-    <visual>
-      <origin
-        xyz="-0.033 0 -0.083"
-        rpy="${pi/2} 0 ${pi/2}" />
-      <geometry>
-        <mesh
-          filename="package://rhr_visualization/meshes/proximal_pad_3.STL" />
-      </geometry>
-      <material
-        name="">
-        <xacro:pad_color/>
-      </material>
-    </visual>
-  </link>
-  <joint
-    name="proximal_3_pad_joint"
-    type="fixed">
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